Commit message: v1

File: ros2_ws/src/amr_description/urdf/robot.urdf (robot description, URDF)
Before this commit: robot amr_description, 10 links, 9 joints
Links:
- removed link camera_depth_link
- removed link camera_depth_link_optical
- removed link camera_rgb_link
- removed link camera_rgb_link_optical
- added link camera_link
Joints:
- removed joint camera_depth_link_jt
- removed joint camera_depth_link_optical_jt
- removed joint camera_rgb_link_jt
- removed joint camera_rgb_link_optical_jt
- added joint camera_joint: type fixed, parent base_link, child camera_link, origin xyz=0.219919 0.038124 0.756912 rpy=0 0 0
- joint laser_frame_jt: origin xyz=0.182324380505574 -2.81953415025293E-05 0.2657 rpy=0 0 0 -> xyz=0.302324380505574 0.0 0.2657 rpy=0 0 0

Commit message: f

File: ros2_ws/src/amr_description/urdf/robot.urdf (robot description, URDF)
Before this commit: robot amr_description, 7 links, 6 joints
Joints:
- joint camera_joint: origin xyz=0.219919 0.038124 0.756912 rpy=0 0 0 -> xyz=0.219919 0.038124 0.79 rpy=0 0.15 0

Commit message: h

File: ros2_ws/src/amr_description/urdf/robot.urdf (robot description, URDF)
Before this commit: robot amr_description, 7 links, 6 joints
Joints:
- joint camera_joint: origin xyz=0.219919 0.038124 0.79 rpy=0 0.15 0 -> xyz=0.219919 0.038124 0.79 rpy=0 0 0
